File: kicad/schematic_all/schematic_all.kicad_sch (KiCad schematic)
At the start: 31 parts, among them J1 Power In, SW1 Button 1, SW2 Encoder 1, SW3 Button 2, SW4 Encoder 2, SW5 Button 3, U2 RPi_Pico, U3 RDA5807M_Module, U4 LM386

Commit message: Added 12V supply + linear regulator to step-down to 5V
Parts:
- removed J1: Power In, TerminalBlock_Phoenix:TerminalBlock_Phoenix_MKDS-1,5-2_1x02_P5.00mm_Horizontal, symbol Connector:USB_B_Micro
- added J1: Barrel_Jack_MountingPin, Connector_BarrelJack:BarrelJack_Horizontal, symbol Connector:Barrel_Jack_MountingPin
- added U1: L7805, Package_TO_SOT_THT:TO-220-3_Vertical, symbol Regulator_Linear:L7805
Connections:
- net +5V: now also U1.3 (OUT); no longer C10.1, U4.6 (V+)
- net GND: now also J1.2, J1.MP (MountPin), U1.2 (GND)
- new net +12V: C10.1, J1.1, U1.1 (IN), U4.6 (V+)
- no-connect marks 19 -> 16

Commit message: Replaced jack with a terminal block
Parts:
- removed J1: Barrel_Jack_MountingPin, Connector_BarrelJack:BarrelJack_Horizontal, symbol Connector:Barrel_Jack_MountingPin
- added J1: Screw_Terminal_01x02, symbol Connector:Screw_Terminal_01x02
- C10: value 10uF -> 680uF; footprint Capacitor_THT:CP_Radial_D5.0mm_P2.00mm -> Capacitor_THT:CP_Radial_D8.0mm_P3.50mm
- C13: footprint Capacitor_THT:CP_Radial_D6.3mm_P2.50mm -> Capacitor_THT:CP_Radial_D8.0mm_P3.50mm
Connections:
- net +12V: now also J1.1 (Pin_1)
- net GND: now also J1.2 (Pin_2)
Changed lines of the file:
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@@
 	)
 	(junction
-		(at 27.94 38.1)
-		(diameter 0)
-		(color 0 0 0 0)
-	)
-	(junction
 		(at 238.76 107.95)
 		(diameter 0)
@@
 	(wire
 		(pts
-			(xy 27.94 36.83) (xy 27.94 38.1)
-		)
-		(stroke
-			(width 0)
-			(type default)
-		)
-	)
-	(wire
-		(pts
 			(xy 95.25 111.76) (xy 95.25 113.03)
 		)
@@
 	(wire
 		(pts
-			(xy 43.18 24.13) (xy 43.18 26.67)
-		)
-		(stroke
-			(width 0)
-			(type default)
-		)
-	)
-	(wire
-		(pts
 			(xy 102.87 119.38) (xy 109.22 119.38)
 		)
@@
 	(wire
 		(pts
-			(xy 44.45 31.75) (xy 44.45 38.1)
-		)
-		(stroke
-			(width 0)
-			(type default)
-		)
-	)
-	(wire
-		(pts
 			(xy 231.14 132.08) (xy 231.14 137.16)
 		)
@@
 	(wire
 		(pts
+			(xy 21.59 31.75) (xy 21.59 25.4)
+		)
+		(stroke
+			(width 0)
+			(type default)
+		)
+	)
+	(wire
+		(pts
+			(xy 21.59 25.4) (xy 26.67 25.4)
+		)
+		(stroke
+			(width 0)
+			(type default)
+		)
+	)
+	(wire
+		(pts
 			(xy 77.47 63.5) (xy 64.77 63.5)
 		)
@@
 	(wire
 		(pts
-			(xy 44.45 38.1) (xy 27.94 38.1)
-		)
-		(stroke
-			(width 0)
-			(type default)
-		)
-	)
-	(wire
-		(pts
 			(xy 49.53 156.21) (xy 52.07 156.21)
 		)
@@
 	(wire
 		(pts
-			(xy 43.18 26.67) (xy 35.56 26.67)
-		)
-		(stroke
-			(width 0)
-			(type default)
-		)
-	)
-	(wire
-		(pts
 			(xy 86.36 121.92) (xy 86.36 111.76)
 		)
@@
 	(wire
 		(pts
-			(xy 27.94 38.1) (xy 27.94 39.37)
-		)
-		(stroke
-			(width 0)
-			(type default)
-		)
-	)
-	(wire
-		(pts
 			(xy 248.92 129.54) (xy 251.46 129.54)
 		)
@@
 	(wire
 		(pts
-			(xy 35.56 31.75) (xy 44.45 31.75)
-		)
-		(stroke
-			(width 0)
-			(type default)
-		)
-	)
-	(wire
-		(pts
 			(xy 257.81 67.31) (xy 257.81 69.85)
 		)
@@
 	(wire
 		(pts
+			(xy 29.21 22.86) (xy 29.21 25.4)
+		)
+		(stroke
+			(width 0)
+			(type default)
+		)
+	)
+	(wire
+		(pts
 			(xy 20.32 58.42) (xy 20.32 60.96)
 		)
@@
 	)
 	(symbol
+		(lib_id "Connector:Screw_Terminal_01x02")
+		(at 29.21 30.48 270)
+		(unit 1)
+		(exclude_from_sim no)
+		(in_bom yes)
+		(on_board yes)
+		(dnp no)
+		(fields_autoplaced yes)
+		(property "Reference" "J1"
+			(at 31.75 29.2099 90)
+			(effects
+				(font
+					(size 1.27 1.27)
+				)
+				(justify left)
+			)
+		)
+		(property "Value" "Screw_Terminal_01x02"
+			(at 31.75 31.7499 90)
+			(effects
+				(font
+					(size 1.27 1.27)
+				)
+				(justify left)
+			)
+		)
+		(property "Footprint" ""
+			(at 29.21 30.48 0)
+			(effects
+				(font
+					(size 1.27 1.27)
+				)
+				(hide yes)
+			)
+		)
+		(property "Datasheet" "~"
+			(at 29.21 30.48 0)
+			(effects
+				(font
+					(size 1.27 1.27)
+				)
+				(hide yes)
+			)
+		)
+		(property "Description" "Generic screw terminal, single row, 01x02, script generated (kicad-library-utils/schlib/autogen/connector/)"
+			(at 29.21 30.48 0)
+			(effects
+				(font
+					(size 1.27 1.27)
+				)
+				(hide yes)
+			)
+		)
+		(pin "1"
+		)
+		(pin "2"
+		)
+		(instances
+			(project ""
+				(path "/017a32bd-a431-4565-87b4-2161296abf15"
+					(reference "J1")
+					(unit 1)
+				)
+			)
+		)
+	)
+	(symbol
 		(lib_id "Mechanical:MountingHole_Pad")
 		(at 58.42 179.07 0)
@@
 	(symbol
 		(lib_id "power:Earth")
-		(at 27.94 39.37 0)
+		(at 21.59 31.75 0)
 		(unit 1)
 		(exclude_from_sim no)
@@
 		(fields_autoplaced yes)
 		(property "Reference" "#PWR01"
-			(at 27.94 45.72 0)
+			(at 21.59 38.1 0)
 			(effects
 				(font
@@
 		)
 		(property "Value" "GND"
-			(at 30.48 40.6399 0)
+			(at 21.59 36.83 0)
 			(effects
 				(font
 					(size 1.27 1.27)
 				)
-				(justify left)
 			)
 		)
 		(property "Footprint" ""
-			(at 27.94 39.37 0)
+			(at 21.59 31.75 0)
 			(effects
 				(font
@@
 		)
 		(property "Datasheet" "~"
-			(at 27.94 39.37 0)
+			(at 21.59 31.75 0)
 			(effects
 				(font
@@
 		)
 		(property "Description" "Power symbol creates a global label with name \"Earth\""
-			(at 27.94 39.37 0)
+			(at 21.59 31.75 0)
 			(effects
 				(font
@@
 	(symbol
 		(lib_id "power:+12V")
-		(at 43.18 24.13 0)
+		(at 29.21 22.86 0)
 		(unit 1)
 		(exclude_from_sim no)
@@
 		(fields_autoplaced yes)
 		(property "Reference" "#PWR03"
-			(at 43.18 27.94 0)
+			(at 29.21 26.67 0)
 			(effects
 				(font
@@
 		)
 		(property "Value" "+12V"
-			(at 43.18 19.05 0)
+			(at 29.21 17.78 0)
 			(effects
 				(font
@@
 		)
 		(property "Footprint" ""
-			(at 43.18 24.13 0)
+			(at 29.21 22.86 0)
 			(effects
 				(font
@@
 		)
 		(property "Datasheet" ""
-			(at 43.18 24.13 0)
+			(at 29.21 22.86 0)
 			(effects
 				(font
@@
 		)
 		(property "Description" "Power symbol creates a global label with name \"+12V\""
-			(at 43.18 24.13 0)
+			(at 29.21 22.86 0)
 			(effects
 				(font
@@
 			)
 		)
-		(property "Value" "10uF"
+		(property "Value" "680uF"
 			(at 245.364 104.14 90)
 			(effects
@@
 			)
 		)
-		(property "Footprint" "Capacitor_THT:CP_Radial_D5.0mm_P2.00mm"
+		(property "Footprint" "Capacitor_THT:CP_Radial_D8.0mm_P3.50mm"
 			(at 245.11 107.95 0)
 			(effects
@@
 	)
 	(symbol
-		(lib_id "Connector:Barrel_Jack_MountingPin")
-		(at 27.94 29.21 0)
-		(unit 1)
-		(exclude_from_sim no)
-		(in_bom yes)
-		(on_board yes)
-		(dnp no)
-		(fields_autoplaced yes)
-		(property "Reference" "J1"
-			(at 27.94 20.32 0)
-			(effects
-				(font
-					(size 1.27 1.27)
-				)
-			)
-		)
-		(property "Value" "Barrel_Jack_MountingPin"
-			(at 27.94 22.86 0)
-			(effects
-				(font
-					(size 1.27 1.27)
-				)
-			)
-		)
-		(property "Footprint" "Connector_BarrelJack:BarrelJack_Horizontal"
-			(at 29.21 30.226 0)
-			(effects
-				(font
-					(size 1.27 1.27)
-				)
-				(hide yes)
-			)
-		)
-		(property "Datasheet" "~"
-			(at 29.21 30.226 0)
-			(effects
-				(font
-					(size 1.27 1.27)
-				)
-				(hide yes)
-			)
-		)
-		(property "Description" "DC Barrel Jack with a mounting pin"
-			(at 27.94 29.21 0)
-			(effects
-				(font
-					(size 1.27 1.27)
-				)
-				(hide yes)
-			)
-		)
-		(pin "1"
-		)
-		(pin "2"
-		)
-		(pin "MP"
-		)
-		(instances
-			(project ""
-				(path "/017a32bd-a431-4565-87b4-2161296abf15"
-					(reference "J1")
-					(unit 1)
-				)
-			)
-		)
-	)
-	(symbol
 		(lib_id "power:+5V")
 		(at 35.56 58.42 0)
@@
 			)
 		)
-		(property "Footprint" "Capacitor_THT:CP_Radial_D6.3mm_P2.50mm"
+		(property "Footprint" "Capacitor_THT:CP_Radial_D8.0mm_P3.50mm"
 			(at 257.81 129.54 0)
 			(effects

Commit message: Minor changes
Parts:
- J1: footprint (none) -> TerminalBlock_Phoenix:TerminalBlock_Phoenix_MKDS-1,5-2_1x02_P5.00mm_Horizontal
Changed lines of the file:
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@@
 			)
 		)
-		(property "Footprint" ""
+		(property "Footprint" "TerminalBlock_Phoenix:TerminalBlock_Phoenix_MKDS-1,5-2_1x02_P5.00mm_Horizontal"
 			(at 29.21 30.48 0)
 			(effects
